File: pcb/main_board/mcu.kicad_sch (KiCad schematic)
At the start: 16 parts

Commit message: Fully annotated board
Signed-off-by: James Hughes <james@pyrosoftsolutions.co.uk>
Parts:
- C1, C2: renamed from C?; footprint (none) -> Capacitor_SMD:C_0402_1005Metric
- C9: renamed from C?; footprint (none) -> Capacitor_SMD:C_0603_1608Metric
- R3: renamed from R?; footprint (none) -> Resistor_SMD:R_0603_1608Metric
- SW1, SW2: renamed from SW?; footprint (none) -> ProjectLib:SW_TS-1187A-B-A-B
- gave numbers to parts that had none: 10
Changed lines of the file:
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@@
   (symbol (lib_id "Device:C_Small") (at 125.216 35.796 0) (unit 1)
     (in_bom yes) (on_board yes)
-    (property "Reference" "C?" (id 0) (at 122.716 34.296 0)
+    (property "Reference" "C4" (id 0) (at 122.716 34.296 0)
       (effects (font (size 1.27 1.27)) (justify left))
     )
@@
   (symbol (lib_id "Switch:SW_Push_Dual") (at 78.232 51.054 90) (unit 1)
     (in_bom yes) (on_board yes)
-    (property "Reference" "SW?" (id 0) (at 71.232 50.474 90)
+    (property "Reference" "SW1" (id 0) (at 71.232 50.474 90)
       (effects (font (size 1.27 1.27)) (justify right))
     )
@@
       (effects (font (size 1.27 1.27)) (justify right))
     )
-    (property "Footprint" "" (id 2) (at 73.152 51.054 0)
+    (property "Footprint" "ProjectLib:SW_TS-1187A-B-A-B" (id 2) (at 73.152 51.054 0)
       (effects (font (size 1.27 1.27)) hide)
     )
@@
   (symbol (lib_id "Device:C_Small") (at 129.216 35.796 0) (unit 1)
     (in_bom yes) (on_board yes)
-    (property "Reference" "C?" (id 0) (at 126.716 34.296 0)
+    (property "Reference" "C5" (id 0) (at 126.716 34.296 0)
       (effects (font (size 1.27 1.27)) (justify left))
     )
@@
   (symbol (lib_id "Device:C_Small") (at 90.932 75.438 0) (unit 1)
     (in_bom yes) (on_board yes)
-    (property "Reference" "C?" (id 0) (at 88.392 73.914 0)
+    (property "Reference" "C1" (id 0) (at 88.392 73.914 0)
       (effects (font (size 1.27 1.27)) (justify left))
     )
@@
       (effects (font (size 1.27 1.27)) (justify left))
     )
-    (property "Footprint" "" (id 2) (at 90.932 75.438 0)
+    (property "Footprint" "Capacitor_SMD:C_0402_1005Metric" (id 2) (at 90.932 75.438 0)
       (effects (font (size 1.27 1.27)) hide)
     )
@@
   (symbol (lib_id "MCU_ST_STM32F0:STM32F072C8Tx") (at 140.716 83.312 0) (unit 1)
     (in_bom yes) (on_board yes) (fields_autoplaced)
-    (property "Reference" "U?" (id 0) (at 145.2754 120.952 0)
+    (property "Reference" "U1" (id 0) (at 145.2754 120.952 0)
       (effects (font (size 1.27 1.27)) (justify left))
     )
@@
   (symbol (lib_id "Device:C_Small") (at 148.216 35.796 0) (unit 1)
     (in_bom yes) (on_board yes)
-    (property "Reference" "C?" (id 0) (at 145.716 34.296 0)
+    (property "Reference" "C9" (id 0) (at 145.716 34.296 0)
       (effects (font (size 1.27 1.27)) (justify left))
     )
@@
       (effects (font (size 0.75 0.75)) (justify left))
     )
-    (property "Footprint" "" (id 2) (at 148.216 35.796 0)
+    (property "Footprint" "Capacitor_SMD:C_0603_1608Metric" (id 2) (at 148.216 35.796 0)
       (effects (font (size 1.27 1.27)) hide)
     )
@@
   (symbol (lib_id "Device:C_Small") (at 157.716 35.796 0) (unit 1)
     (in_bom yes) (on_board yes)
-    (property "Reference" "C?" (id 0) (at 155.216 34.296 0)
+    (property "Reference" "C11" (id 0) (at 155.216 34.296 0)
       (effects (font (size 1.27 1.27)) (justify left))
     )
@@
   (symbol (lib_id "Device:C_Small") (at 114.162 47.244 0) (unit 1)
     (in_bom yes) (on_board yes)
-    (property "Reference" "C?" (id 0) (at 111.662 45.744 0)
+    (property "Reference" "C3" (id 0) (at 111.662 45.744 0)
       (effects (font (size 1.27 1.27)) (justify left))
     )
@@
   (symbol (lib_id "Device:C_Small") (at 100.838 82.804 0) (unit 1)
     (in_bom yes) (on_board yes)
-    (property "Reference" "C?" (id 0) (at 101.346 81.026 0)
+    (property "Reference" "C2" (id 0) (at 101.346 81.026 0)
       (effects (font (size 1.27 1.27)) (justify left))
     )
@@
       (effects (font (size 1.27 1.27)) (justify left))
     )
-    (property "Footprint" "" (id 2) (at 100.838 82.804 0)
+    (property "Footprint" "Capacitor_SMD:C_0402_1005Metric" (id 2) (at 100.838 82.804 0)
       (effects (font (size 1.27 1.27)) hide)
     )
@@
   (symbol (lib_id "Device:R_Small") (at 78.232 62.23 0) (unit 1)
     (in_bom yes) (on_board yes) (fields_autoplaced)
-    (property "Reference" "R?" (id 0) (at 80.822 60.9599 0)
+    (property "Reference" "R3" (id 0) (at 80.822 60.9599 0)
       (effects (font (size 1.27 1.27)) (justify left))
     )
@@
       (effects (font (size 1.27 1.27)) (justify left))
     )
-    (property "Footprint" "" (id 2) (at 78.232 62.23 0)
+    (property "Footprint" "Resistor_SMD:R_0603_1608Metric" (id 2) (at 78.232 62.23 0)
       (effects (font (size 1.27 1.27)) hide)
     )
@@
   (symbol (lib_id "Switch:SW_Push_Dual") (at 89.408 44.958 90) (unit 1)
     (in_bom yes) (on_board yes) (fields_autoplaced)
-    (property "Reference" "SW?" (id 0) (at 95.778 43.6879 90)
+    (property "Reference" "SW2" (id 0) (at 95.778 43.6879 90)
       (effects (font (size 1.27 1.27)) (justify right))
     )
@@
       (effects (font (size 1.27 1.27)) (justify right))
     )
-    (property "Footprint" "" (id 2) (at 84.328 44.958 0)
+    (property "Footprint" "ProjectLib:SW_TS-1187A-B-A-B" (id 2) (at 84.328 44.958 0)
       (effects (font (size 1.27 1.27)) hide)
     )
@@
   (symbol (lib_id "Device:C_Small") (at 153.716 35.796 0) (unit 1)
     (in_bom yes) (on_board yes)
-    (property "Reference" "C?" (id 0) (at 151.216 34.296 0)
+    (property "Reference" "C10" (id 0) (at 151.216 34.296 0)
       (effects (font (size 1.27 1.27)) (justify left))
     )
@@
   (symbol (lib_id "Device:Crystal_GND24_Small") (at 94.742 79.248 180) (unit 1)
     (in_bom yes) (on_board yes)
-    (property "Reference" "Y?" (id 0) (at 91.694 81.534 0))
+    (property "Reference" "Y1" (id 0) (at 91.694 81.534 0))
     (property "Value" "Crystal_GND24_Small" (id 1) (at 84.582 83.566 0))
     (property "Footprint" "Crystal:Crystal_SMD_3225-4Pin_3.2x2.5mm" (id 2) (at 94.742 79.248 0)
@@
   (symbol (lib_id "Device:C_Small") (at 138.716 35.796 0) (unit 1)
     (in_bom yes) (on_board yes)
-    (property "Reference" "C?" (id 0) (at 136.216 34.296 0)
+    (property "Reference" "C7" (id 0) (at 136.216 34.296 0)
       (effects (font (size 1.27 1.27)) (justify left))
     )
@@
   (symbol (lib_id "Device:C_Small") (at 134.716 35.796 0) (unit 1)
     (in_bom yes) (on_board yes)
-    (property "Reference" "C?" (id 0) (at 132.216 34.296 0)
+    (property "Reference" "C6" (id 0) (at 132.216 34.296 0)
       (effects (font (size 1.27 1.27)) (justify left))
     )
@@
   (symbol (lib_id "Device:C_Small") (at 144.216 35.796 0) (unit 1)
     (in_bom yes) (on_board yes)
-    (property "Reference" "C?" (id 0) (at 141.716 34.296 0)
-      (effects (font (size 1.27 1.27)) (justify left))
-    )
+    (property "Reference" "C8" (id 0) (at 141.716 34.296 0)
+      (effects (font (size 1.27 1.27)) (justify left))
+    )
