File: pcb/main_board/pwr_cnd.kicad_sch (KiCad schematic)
At the start: 3 parts

Commit message: Fully annotated board
Signed-off-by: James Hughes <james@pyrosoftsolutions.co.uk>
Parts:
- C12: renamed from C?; footprint (none) -> Capacitor_SMD:C_0603_1608Metric
- J2: renamed from J?; footprint (none) -> Connector_PinHeader_2.54mm:PinHeader_1x02_P2.54mm_Vertical
- gave numbers to parts that had none: 1
Changed lines of the file:
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@@
   (symbol (lib_id "Connector:Conn_01x02_Female") (at 142.748 98.298 0) (unit 1)
     (in_bom yes) (on_board yes) (fields_autoplaced)
-    (property "Reference" "J?" (id 0) (at 143.51 98.2979 0)
+    (property "Reference" "J2" (id 0) (at 143.51 98.2979 0)
       (effects (font (size 1.27 1.27)) (justify left))
     )
@@
       (effects (font (size 1.27 1.27)) (justify left))
     )
-    (property "Footprint" "" (id 2) (at 142.748 98.298 0)
+    (property "Footprint" "Connector_PinHeader_2.54mm:PinHeader_1x02_P2.54mm_Vertical" (id 2) (at 142.748 98.298 0)
       (effects (font (size 1.27 1.27)) hide)
     )
@@
   (symbol (lib_id "Regulator_Linear:XC6206PxxxMR") (at 109.22 91.186 0) (unit 1)
     (in_bom yes) (on_board yes) (fields_autoplaced)
-    (property "Reference" "U?" (id 0) (at 109.22 83.82 0))
+    (property "Reference" "U2" (id 0) (at 109.22 83.82 0))
     (property "Value" "XC6206PxxxMR" (id 1) (at 109.22 86.36 0))
     (property "Footprint" "Package_TO_SOT_SMD:SOT-23" (id 2) (at 109.22 85.471 0)
@@
   (symbol (lib_id "Device:C_Small") (at 122.174 96.012 0) (unit 1)
     (in_bom yes) (on_board yes) (fields_autoplaced)
-    (property "Reference" "C?" (id 0) (at 125.73 94.7482 0)
+    (property "Reference" "C12" (id 0) (at 125.73 94.7482 0)
       (effects (font (size 1.27 1.27)) (justify left))
     )
@@
       (effects (font (size 1.27 1.27)) (justify left))
     )
-    (property "Footprint" "" (id 2) (at 122.174 96.012 0)
+    (property "Footprint" "Capacitor_SMD:C_0603_1608Metric" (id 2) (at 122.174 96.012 0)
       (effects (font (size 1.27 1.27)) hide)
     )
