File: pcb/main_board/usb_in.kicad_sch (KiCad schematic)
At the start: 3 parts

Commit message: Fully annotated board
Signed-off-by: James Hughes <james@pyrosoftsolutions.co.uk>
Parts:
- R1, R2: renamed from R?; footprint (none) -> Resistor_SMD:R_0603_1608Metric
- gave numbers to parts that had none: 1
Changed lines of the file:
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@@
   (symbol (lib_id "Device:R_Small") (at 109.728 81.28 90) (unit 1)
     (in_bom yes) (on_board yes)
-    (property "Reference" "R?" (id 0) (at 109.728 77.724 90))
+    (property "Reference" "R1" (id 0) (at 109.728 77.724 90))
     (property "Value" "5.1k" (id 1) (at 109.728 79.502 90))
-    (property "Footprint" "" (id 2) (at 109.728 81.28 0)
+    (property "Footprint" "Resistor_SMD:R_0603_1608Metric" (id 2) (at 109.728 81.28 0)
       (effects (font (size 1.27 1.27)) hide)
     )
@@
   (symbol (lib_id "Connector:USB_C_Receptacle_USB2.0") (at 90.17 91.44 0) (unit 1)
     (in_bom yes) (on_board yes) (fields_autoplaced)
-    (property "Reference" "J?" (id 0) (at 90.17 68.58 0))
+    (property "Reference" "J1" (id 0) (at 90.17 68.58 0))
     (property "Value" "USB_C_Receptacle_USB2.0" (id 1) (at 90.17 71.12 0))
     (property "Footprint" "Connector_USB:USB_C_Receptacle_HRO_TYPE-C-31-M-12" (id 2) (at 93.98 91.44 0)
@@
   (symbol (lib_id "Device:R_Small") (at 109.728 83.82 90) (unit 1)
     (in_bom yes) (on_board yes)
-    (property "Reference" "R?" (id 0) (at 109.728 85.598 90))
+    (property "Reference" "R2" (id 0) (at 109.728 85.598 90))
     (property "Value" "5.1kR" (id 1) (at 109.728 87.376 90))
-    (property "Footprint" "" (id 2) (at 109.728 83.82 0)
+    (property "Footprint" "Resistor_SMD:R_0603_1608Metric" (id 2) (at 109.728 83.82 0)
       (effects (font (size 1.27 1.27)) hide)
     )
